File: pcb/Atreus62.kicad_pcb (KiCad board)
At the start: 2 copper layers, 270.1 x 112.9 mm, 126 parts, among them SW1 SWITCH_PUSH, SW10 SWITCH_PUSH, SW11 SWITCH_PUSH, SW12 SWITCH_PUSH, SW13 SWITCH_PUSH, SW14 SWITCH_PUSH, SW15 SWITCH_PUSH, SW16 SWITCH_PUSH, SW17 SWITCH_PUSH, SW18 SWITCH_PUSH, SW19 SWITCH_PUSH, SW2 SWITCH_PUSH, SW20 SWITCH_PUSH, SW21 SWITCH_PUSH, SW22 SWITCH_PUSH, SW23 SWITCH_PUSH, SW24 SWITCH_PUSH, SW25 SWITCH_PUSH, SW26 SWITCH_PUSH, SW27 SWITCH_PUSH, SW28 SWITCH_PUSH, SW29 SWITCH_PUSH, SW3 SWITCH_PUSH, SW30 SWITCH_PUSH, SW31 SWITCH_PUSH, SW32 SWITCH_PUSH, SW33 SWITCH_PUSH, SW34 SWITCH_PUSH, SW35 SWITCH_PUSH, SW36 SWITCH_PUSH, SW37 SWITCH_PUSH, SW38 SWITCH_PUSH, SW39 SWITCH_PUSH, SW4 SWITCH_PUSH, SW40 SWITCH_PUSH, SW41 SWITCH_PUSH, SW42 SWITCH_PUSH, SW43 SWITCH_PUSH, SW44 SWITCH_PUSH, SW45 SWITCH_PUSH, SW46 SWITCH_PUSH, SW47 SWITCH_PUSH, SW48 SWITCH_PUSH, SW49 SWITCH_PUSH, SW5 SWITCH_PUSH, SW50 SWITCH_PUSH, SW51 SWITCH_PUSH, SW52 SWITCH_PUSH, SW53 SWITCH_PUSH, SW54 SWITCH_PUSH, SW55 SWITCH_PUSH, SW56 SWITCH_PUSH, SW57 SWITCH_PUSH, SW58 SWITCH_PUSH, SW59 SWITCH_PUSH, SW6 SWITCH_PUSH, SW60 SWITCH_PUSH, SW61 SWITCH_PUSH, SW62 SWITCH_PUSH, SW7 SWITCH_PUSH, SW8 SWITCH_PUSH, SW9 SWITCH_PUSH, U1 ARDUINO_PRO_MICRO

Commit message: Updated
updated pcb design files
Other:
- board text added: "atreus62 design by profet23 : GPLv3"
Changed lines of the file:
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@@
-(kicad_pcb (version 20171130) (host pcbnew "(5.1.4-0)")
+(kicad_pcb (version 20171130) (host pcbnew "(5.1.4)-1")
   (general
     (thickness 1.6)
-    (drawings 1257)
+    (drawings 1258)
     (tracks 1028)
     (zones 0)
@@
     (39 F.Mask user)
     (40 Dwgs.User user hide)
-    (41 Cmts.User user hide)
+    (41 Cmts.User user)
     (42 Eco1.User user hide)
     (43 Eco2.User user hide)
@@
       (net 84 "Net-(SW-RST1-Pad2)"))
   )
+  (gr_text "atreus62 design by profet23 : GPLv3" (at 223.653858 43.791457) (layer F.SilkS)
+    (effects (font (size 1.5 1.5) (thickness 0.3)))
+  )
   (gr_text "Made Compatible by NaCly" (at 189.363858 43.791457) (layer F.SilkS)

Commit message: updated to license is easier to read.
updated to license is easier to read.
Other:
- board text added: "GPLv3"
- board text added: "profet23"
Changed lines of the file:
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@@
   (general
     (thickness 1.6)
-    (drawings 1258)
+    (drawings 1261)
     (tracks 1028)
     (zones 0)
@@
       (net 84 "Net-(SW-RST1-Pad2)"))
   )
+  (gr_text profet23 (at 148.723858 121.515457) (layer F.SilkS)
+    (effects (font (size 25 25) (thickness 3)))
+  )
+  (gr_text GPLv3 (at 214.509858 75.541457) (layer F.SilkS)
+    (effects (font (size 25 25) (thickness 3)))
+  )
+  (gr_text GPLv3 (at 77.857858 78.335457) (layer F.SilkS)
+    (effects (font (size 25 25) (thickness 3)))
+  )
   (gr_text "atreus62 design by profet23 : GPLv3" (at 223.653858 43.791457) (layer F.SilkS)

Commit message: .
.
Other:
- board text added: "atreus62 design by profet23 : GPLv3 based on atreus by Phil Hagelberg"
- board text removed: "GPLv3"
- board text removed: "atreus62 design by profet23 : GPLv3"
- board text removed: "profet23"
Changed lines of the file:
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@@
   (general
     (thickness 1.6)
-    (drawings 1261)
+    (drawings 1258)
     (tracks 1028)
     (zones 0)
@@
       (net 84 "Net-(SW-RST1-Pad2)"))
   )
-  (gr_text profet23 (at 148.723858 121.515457) (layer F.SilkS)
-    (effects (font (size 25 25) (thickness 3)))
-  )
-  (gr_text GPLv3 (at 214.509858 75.541457) (layer F.SilkS)
-    (effects (font (size 25 25) (thickness 3)))
-  )
-  (gr_text GPLv3 (at 77.857858 78.335457) (layer F.SilkS)
-    (effects (font (size 25 25) (thickness 3)))
-  )
-  (gr_text "atreus62 design by profet23 : GPLv3" (at 223.653858 43.791457) (layer F.SilkS)
+  (gr_text "Made Compatible by NaCly" (at 100.971858 42.775457) (layer F.SilkS)
     (effects (font (size 1.5 1.5) (thickness 0.3)))
   )
-  (gr_text "Made Compatible by NaCly" (at 189.363858 43.791457) (layer F.SilkS)
-    (effects (font (size 1 1) (thickness 0.15)))
+  (gr_text "atreus62 design by profet23 : GPLv3\nbased on atreus by Phil Hagelberg" (at 200.793858 43.791457) (layer F.SilkS)
+    (effects (font (size 1.5 1.5) (thickness 0.3)))
   )
   (gr_text atreus62 (at 148.34 126.44) (layer B.SilkS)
